File: Planar_Flyback_PSU/Planar_Flyback_PSU.kicad_sch (KiCad schematic)
At the start: 0 parts

Commit message: update repo
Parts:
- added C1, C2, C42: C_Polarized, symbol Device:C_Polarized
- added C10, C14, C15, C16, C19, C32: 1u, symbol Device:C
- added C11, C12, C21, C22, C23, C24, C27, C28, C29, C30, C31, C39, C40, C41: 10u, Capacitor_SMD:C_0805_2012Metric, symbol Device:C
- added C13, C25, C26, C33, C34, C35, C36, C5, C6, C7, C8, C9: C_Polarized, Capacitor_Tantalum_SMD:CP_EIA-3528-12_Kemet-T, symbol Device:C_Polarized
- added C17, C18, C20: 100n, Capacitor_SMD:C_0603_1608Metric, symbol Device:C
- added C3, C38, C4, C43, C44: C, symbol Device:C
- added C37: 100n, symbol Device:C
- added D1, D2: MDB6S, Package_SO:TSSOP-4_4.4x5mm_P4mm, symbol Diode_Bridge:MDB6S
- added D32, D33, D34, D35, D36: D_Schottky, Diode_SMD:D_SOD-128, symbol Device:D_Schottky
- added D4, D5, D6, D7, D8: YLED1206R, LED_SMD:LED_1206_3216Metric, symbol Device:LED
- added F1: Fuse, symbol Device:Fuse
- added IC1: NCP1342AMDCDAD1R2G, Library:NCP1342AMDCDAD1R2G, symbol NCP1342AMDCDAD1R2G:NCP1342AMDCDAD1R2G
- added IC2: CD4044BPWR, Library:SOP65P640X120-16N, symbol CD4044BPWR:CD4044BPWR
- added J1: IEC_60320_C14_Receptacle, symbol Connector:IEC_60320_C14_Receptacle
- added JP1, JP2, JP3, JP4: SolderJumper_2_Bridged, Jumper:SolderJumper-2_P1.3mm_Bridged2Bar_RoundedPad1.0x1.5mm, symbol Jumper:SolderJumper_2_Bridged
- added L1: L_Ferrite_Coupled, symbol Device:L_Ferrite_Coupled
- added L2, L3: 12uH, Inductor_SMD:L_Coilcraft_XAL6020-XXX, symbol Device:L
- added L4, L5: l, Inductor_SMD:L_Coilcraft_XAL6020-XXX, symbol Device:L
- added Q1, Q3, Q4: BSC072N08NS5, Package_TO_SOT_SMD:TDSON-8-1, symbol Transistor_FET:BSC072N08NS5
- added Q5: 2N7002, Package_TO_SOT_SMD:SOT-23, symbol Transistor_FET:2N7002
- added R1, R10, R2, R21, R22, R3, R4, R5, R6: R, symbol Device:R
- added R11, R12, R14, R20, R8: 10k, symbol Device:R
- added R13: 5k1, symbol Device:R
- added R15, R16: 100R, symbol Device:R
- added R17, R18, R19, R7, R9: 1k, symbol Device:R
- added R29, R30, R31, R32, R33, R38, R40, R41, R44, R46, R47, R48, R49: R, Resistor_SMD:R_0603_1608Metric, symbol Device:R
- added R34, R36, R37, R39: 220R, Resistor_SMD:R_0805_2012Metric, symbol Device:R
- added R35: 2k, Resistor_SMD:R_0805_2012Metric, symbol Device:R
- added R42: 100k, Resistor_SMD:R_0603_1608Metric, symbol Device:R
- added R43: 3k3, Resistor_SMD:R_0603_1608Metric, symbol Device:R
- added R50: 2R, Resistor_SMD:R_0603_1608Metric, symbol Device:R
- added T1: Transformer_1P_2S, symbol Device:Transformer_1P_2S
- added U10: TLP291, Package_SO:SOIC-4_4.55x2.6mm_P1.27mm, symbol Isolator:TLP291
- added U11, U12: AMS1117-3.3, Package_TO_SOT_SMD:SOT-223-3_TabPin2, symbol Regulator_Linear:AMS1117-3.3
- added U2, U3: LM358, symbol Amplifier_Operational:LM358
- added U4, U5: LM393, symbol Comparator:LM393
- added U7, U8: LV2842XLVDDCR, Package_TO_SOT_SMD:SOT-23-6, symbol Regulator_Switching:LV2862XDDC
- added U9: NCP4306, Package_SO:SOIC-8_3.9x4.9mm_P1.27mm, symbol Regulator_Controller:NCP4308AD
Connections:
- new net: C23.1, C26.1, C9.1, U12.2 (VO)
- new net: R11.2, R16.1, U3.5 (+)
- new net: C37.1, R12.1, U3.7, U4.6 (-)
- new net: R12.2, R15.1, U3.6 (-)
- new net: C3.1, F1.2, L1.1
- new net: C3.2, J1.2 (N), L1.3
- new net: R18.2, R9.1, U3.3 (+)
- new net: Q5.1 (G), R8.2
- new net: D5.2 (A), R35.2
- new net: C10.1, R5.1, R6.2, U4.5 (+)
- new net: Q1.5 (D), R16.2, R29.1, R4.1
- new net: R29.2, R30.1, U7.3 (FB)
- new net: R20.1, U3.1
- new net: R17.1, R19.2, R20.2, U3.2 (-)
- new net: C1.1, D1.1 (+), L5.1
- new net: F1.1, J1.1 (L)
- new net: C22.1, C7.1, C8.1, L3.2
- new net: C17.2, D32.1 (K), L2.1, U7.6 (SW)
- new net: C21.1, C5.1, C6.1, L2.2, R15.2, R4.2
- new net: D8.2 (A), R39.1
- new net: C2.1, C38.1, L5.2, R41.2, T1.6 (SD)
- new net: IC1.5 (CS), Q4.1 (S), Q4.2 (S), Q4.3 (S), R10.1
- new net: D36.1 (K), IC1.4 (ZCD/OPP), R48.1, R49.2
- new net: D36.2 (A), R47.1, R48.2
- new net: R31.2, R32.1, U8.3 (FB)
- new net: L4.1, Q1.1 (S), Q1.2 (S), Q1.3 (S)
- new net: C29.1, C30.1, C31.1, L4.2, R34.1
- new net: C4.2, D1.3, D2.3, L1.4
- new net: C4.1, D1.4, D2.4, L1.2
- new net: D34.1 (K), R40.1
- new net: D34.2 (A), Q4.5 (D), T1.5 (SC)
- new net: C42.1, C43.1, D35.1 (K), IC1.8 (VCC)
- new net: R3.2, R9.2
- new net: D7.2 (A), R37.1
- new net: IC1.7 (DRV), Q4.4 (G), R42.1
- new net: C18.2, D33.1 (K), L3.1, U8.6 (SW)
- new net: R17.2, R3.1
- new net: C44.1, U10.2
- new net: C44.2, R22.2
- new net: R44.1, U9.2 (MIN_TOFF)
- new net: R43.1, U9.3 (MIN_TON)
- new net: Q3.5 (D), T1.1 (AA), U9.6 (CS)
- new net: R50.2, U9.8 (DRV)
- new net: C17.1, U7.1 (CB)
- new net: C11.1, JP1.1 (A), U7.5 (VIN)
- new net: C28.1, JP3.1 (A), U12.3 (VI)
- new net: IC1.2 (FMAX), R46.2
- new net: D4.2 (A), R34.2
- new net: Q3.4 (G), R50.1
- new net: IC1.9 (HV), R38.2
- new net: C38.2, R40.2, R41.1
- new net: C27.1, JP4.1 (A), U11.3 (VI)
- new net: R21.1, R22.1
- new net: C18.1, U8.1 (CB)
- new net: C12.1, JP2.1 (A), U8.5 (VIN)
- new net: C32.1, Q1.4 (G), Q5.3 (D), R13.1, R14.2
- new net: R21.2, U10.1
- new net: R7.1, U4.7
- new net: R33.2, R38.1
- new net: D6.2 (A), R36.2
- new net: D2.1 (+), R33.1
- new net +24V: C14.1, C15.1, C16.1, C19.1, C33.1, C34.1, C35.1, C36.1, C39.1, C40.1, C41.1, JP1.2 (B), JP2.2 (B), JP3.2 (B), JP4.2 (B), R13.2, T1.2 (AB), U2.8 (V+), U3.8 (V+), U4.8 (V+), U5.8 (V+), U9.1 (VCC)
- new net 3v3stb: C13.1, C24.1, C25.1, IC2.16 (VDD), R36.1, R5.2, R7.2, U11.2 (VO)
- new net AUX: D35.2 (A), R47.2, T1.4 (SB)
- new net FB: C20.2, IC1.3 (FB), U10.4
- new net GND: C10.2, C11.2, C12.2, C13.2, C14.2, C15.2, C16.2, C19.2, C21.2, C22.2, C23.2, C24.2, C25.2, C26.2, C27.2, C28.2, C29.2, C30.2, C31.2, C32.2, C33.2, C34.2, C35.2, C36.2, C37.2, C39.2, C40.2, C41.2, C5.2, C6.2, C7.2, C8.2, C9.2, D32.2 (A), D33.2 (A), D4.1 (K), D5.1 (K), D6.1 (K), D7.1 (K), D8.1 (K), IC2.8 (VSS), Q3.1 (S), Q3.2 (S), Q3.3 (S), Q5.2 (S), R11.1, R14.1, R18.1, R19.1, R30.2, R32.2, R43.2, R44.2, R6.1, R8.1, T1.3 (SA), U11.1 (GND), U12.1 (GND), U2.4 (V-), U3.4 (V-), U4.4 (V-), U5.4 (V-), U7.2 (GND), U8.2 (GND), U9.4 (TRIG), U9.7 (GND)
- new net GNDS: C1.2, C2.2, C20.1, C42.2, C43.2, D1.2 (-), IC1.6 (GND), R10.2, R42.2, R46.1, R49.1, U10.3
- no-connect marks 0 -> 3
Other:
- note added: "1206"
- note added: "12V"
- note added: "2512"
- note added: "3V3"
- note added: "3V3a"
- note added: "3V3stb"
- note added: "?????"
- note added: "latch"
- note added: "powerup blanking? softstart by making r10 large or adding c"
- note added: "psu good sig?"
- note added: "shunt"
